File: BKR01AT/BKR01AT.sch (KiCad schematic (older format))
At the start: 46 parts

Commit message: organizando o esquemático
Parts:
- gave numbers to parts that had none: 46
Connections:
- net b_ON_OFF renamed led_ON_OFF
- net b_TEMP renamed led_TEMP
- net b_VIB renamed led_VIB
- net led_F1 renamed b_F1
- net led_F2 renamed b_F2
- net led_RST renamed b_RST
Other:
- note added: "Acelerômetro"
- note added: "Alimentação"
- note added: "Antena"
- note added: "Botões"
- note added: "LEDs"
- note added: "MCU (circuito principal)"
- note added: "TagConnect"
- moved on the sheet: BT1, BT2, C1, C10, C11, C12, C13, C14, C16, C17, C2, C3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

Commit message: LEDs
ajustadadas as resistências pros LEDs e pros botões
Parts:
- R1, R2, R3: value ? -> 100Ω
- R4, R5, R6: value ? -> 10kΩ
Changed lines of the file:
@@
 P 9650 4840
 F 0 "R4" H 9718 4886 50  0000 L CNN
-F 1 "?" H 9718 4795 50  0000 L CNN
+F 1 "10kΩ" H 9718 4795 50  0000 L CNN
 F 2 "" H 9650 4840 50  0001 C CNN
 F 3 "~" H 9650 4840 50  0001 C CNN
@@
 P 8880 4860
 F 0 "R6" H 8948 4906 50  0000 L CNN
-F 1 "?" H 8948 4815 50  0000 L CNN
+F 1 "10kΩ" H 8948 4815 50  0000 L CNN
 F 2 "" H 8880 4860 50  0001 C CNN
 F 3 "~" H 8880 4860 50  0001 C CNN
@@
 P 8055 4845
 F 0 "R5" H 8123 4891 50  0000 L CNN
-F 1 "?" H 8123 4800 50  0000 L CNN
+F 1 "10kΩ" H 8123 4800 50  0000 L CNN
 F 2 "" H 8055 4845 50  0001 C CNN
 F 3 "~" H 8055 4845 50  0001 C CNN
@@
 P 8805 2925
 F 0 "R2" H 8873 2971 50  0000 L CNN
-F 1 "?" H 8873 2880 50  0000 L CNN
+F 1 "100Ω" H 8873 2880 50  0000 L CNN
 F 2 "" H 8805 2925 50  0001 C CNN
 F 3 "~" H 8805 2925 50  0001 C CNN
@@
 P 8065 2950
 F 0 "R3" H 8133 2996 50  0000 L CNN
-F 1 "?" H 8133 2905 50  0000 L CNN
+F 1 "100Ω" H 8133 2905 50  0000 L CNN
 F 2 "" H 8065 2950 50  0001 C CNN
 F 3 "~" H 8065 2950 50  0001 C CNN
@@
 P 9615 2910
 F 0 "R1" H 9683 2956 50  0000 L CNN
-F 1 "?" H 9683 2865 50  0000 L CNN
+F 1 "100Ω" H 9683 2865 50  0000 L CNN
 F 2 "" H 9615 2910 50  0001 C CNN
 F 3 "~" H 9615 2910 50  0001 C CNN

Commit message: BOM
Parts:
- AE1: Part Number (none) -> 2450AT18B100E
- BT1, BT2: Part Number (none) -> CR2032R-HE1
- C1: value 1.0uF -> 1uF
- C16: value C_Small -> 10uF
- C17, C7: value C_Small -> 100nF
- D1: value LED -> Green LED; Part Number (none) -> 150060VS75000
- D2: value LED -> Red LED; Part Number (none) -> 150060VS75000
- D3: value LED -> Red LED; Part Number (none) -> 150060RS75000
- MCU1: Part Number (none) -> nRF52832-QFAB-R
- R1, R2, R3: value 100Ω -> 100; footprint (none) -> Resistor_SMD:R_0402_1005Metric
- R4, R5, R6: value 10kΩ -> 10k; footprint (none) -> Resistor_SMD:R_0402_1005Metric
- SW1, SW2, SW3: Part Number (none) -> PTS636 SL43 LFS
- U1: Part Number (none) -> LIS2DHTR
Changed lines of the file:
@@
 P 3555 1430
 F 0 "C1" H 3463 1384 50  0000 R CNN
-F 1 "1.0uF" H 3463 1475 50  0000 R CNN
+F 1 "1uF" H 3463 1475 50  0000 R CNN
 F 2 "" H 3555 1430 50  0001 C CNN
 F 3 "~" H 3555 1430 50  0001 C CNN
@@
 P 4855 2480
 F 0 "C7" H 4947 2526 50  0000 L CNN
-F 1 "C_Small" H 4947 2435 50  0000 L CNN
+F 1 "100nF" H 4947 2435 50  0000 L CNN
 F 2 "" H 4855 2480 50  0001 C CNN
 F 3 "~" H 4855 2480 50  0001 C CNN
@@
 P 9650 4840
 F 0 "R4" H 9718 4886 50  0000 L CNN
-F 1 "10kΩ" H 9718 4795 50  0000 L CNN
-F 2 "" H 9650 4840 50  0001 C CNN
+F 1 "10k" H 9718 4795 50  0000 L CNN
+F 2 "Resistor_SMD:R_0402_1005Metric" H 9650 4840 50  0001 C CNN
 F 3 "~" H 9650 4840 50  0001 C CNN
 	1    9650 4840
@@
 F 2 "" H 9650 5445 50  0001 C CNN
 F 3 "~" H 9650 5445 50  0001 C CNN
+F 4 "PTS636 SL43 LFS" H 9650 5245 50  0001 C CNN "Part Number"
 	1    9650 5245
 	0    1    1    0
@@
 P 8880 4860
 F 0 "R6" H 8948 4906 50  0000 L CNN
-F 1 "10kΩ" H 8948 4815 50  0000 L CNN
-F 2 "" H 8880 4860 50  0001 C CNN
+F 1 "10k" H 8948 4815 50  0000 L CNN
+F 2 "Resistor_SMD:R_0402_1005Metric" H 8880 4860 50  0001 C CNN
 F 3 "~" H 8880 4860 50  0001 C CNN
 	1    8880 4860
@@
 F 2 "" H 8880 5465 50  0001 C CNN
 F 3 "~" H 8880 5465 50  0001 C CNN
+F 4 "PTS636 SL43 LFS" H 8880 5265 50  0001 C CNN "Part Number"
 	1    8880 5265
 	0    1    1    0
@@
 P 8055 4845
 F 0 "R5" H 8123 4891 50  0000 L CNN
-F 1 "10kΩ" H 8123 4800 50  0000 L CNN
-F 2 "" H 8055 4845 50  0001 C CNN
+F 1 "10k" H 8123 4800 50  0000 L CNN
+F 2 "Resistor_SMD:R_0402_1005Metric" H 8055 4845 50  0001 C CNN
 F 3 "~" H 8055 4845 50  0001 C CNN
 	1    8055 4845
@@
 F 2 "" H 8055 5450 50  0001 C CNN
 F 3 "~" H 8055 5450 50  0001 C CNN
+F 4 "PTS636 SL43 LFS" H 8055 5250 50  0001 C CNN "Part Number"
 	1    8055 5250
 	0    1    1    0
@@
 P 8805 2925
 F 0 "R2" H 8873 2971 50  0000 L CNN
-F 1 "100Ω" H 8873 2880 50  0000 L CNN
-F 2 "" H 8805 2925 50  0001 C CNN
+F 1 "100" H 8873 2880 50  0000 L CNN
+F 2 "Resistor_SMD:R_0402_1005Metric" H 8805 2925 50  0001 C CNN
 F 3 "~" H 8805 2925 50  0001 C CNN
 	1    8805 2925
@@
 P 8805 3235
 F 0 "D2" V 8752 3313 50  0000 L CNN
-F 1 "LED" V 8843 3313 50  0000 L CNN
+F 1 "Red LED" V 8843 3313 50  0000 L CNN
 F 2 "" H 8805 3235 50  0001 C CNN
 F 3 "~" H 8805 3235 50  0001 C CNN
+F 4 "150060VS75000" H 8805 3235 50  0001 C CNN "Part Number"
 	1    8805 3235
 	0    -1   -1   0
@@
 P 8065 2950
 F 0 "R3" H 8133 2996 50  0000 L CNN
-F 1 "100Ω" H 8133 2905 50  0000 L CNN
-F 2 "" H 8065 2950 50  0001 C CNN
+F 1 "100" H 8133 2905 50  0000 L CNN
+F 2 "Resistor_SMD:R_0402_1005Metric" H 8065 2950 50  0001 C CNN
 F 3 "~" H 8065 2950 50  0001 C CNN
 	1    8065 2950
@@
 P 8065 3260
 F 0 "D3" V 8012 3338 50  0000 L CNN
-F 1 "LED" V 8103 3338 50  0000 L CNN
+F 1 "Red LED" V 8103 3338 50  0000 L CNN
 F 2 "" H 8065 3260 50  0001 C CNN
 F 3 "~" H 8065 3260 50  0001 C CNN
+F 4 "150060RS75000" H 8065 3260 50  0001 C CNN "Part Number"
 	1    8065 3260
 	0    -1   -1   0
@@
 P 9615 2910
 F 0 "R1" H 9683 2956 50  0000 L CNN
-F 1 "100Ω" H 9683 2865 50  0000 L CNN
-F 2 "" H 9615 2910 50  0001 C CNN
+F 1 "100" H 9683 2865 50  0000 L CNN
+F 2 "Resistor_SMD:R_0402_1005Metric" H 9615 2910 50  0001 C CNN
 F 3 "~" H 9615 2910 50  0001 C CNN
 	1    9615 2910
@@
 P 9615 3220
 F 0 "D1" V 9562 3298 50  0000 L CNN
-F 1 "LED" V 9653 3298 50  0000 L CNN
+F 1 "Green LED" V 9653 3298 50  0000 L CNN
 F 2 "" H 9615 3220 50  0001 C CNN
 F 3 "~" H 9615 3220 50  0001 C CNN
+F 4 "150060VS75000" H 9615 3220 50  0001 C CNN "Part Number"
 	1    9615 3220
 	0    -1   -1   0
@@
 P 5830 6840
 F 0 "C17" V 5700 6840 50  0000 C CNN
-F 1 "C_Small" V 5630 6840 50  0000 C CNN
+F 1 "100nF" V 5630 6840 50  0000 C CNN
 F 2 "" H 5830 6840 50  0001 C CNN
 F 3 "~" H 5830 6840 50  0001 C CNN
@@
 P 5820 6505
 F 0 "C16" V 5690 6505 50  0000 C CNN
-F 1 "C_Small" V 5620 6505 50  0000 C CNN
+F 1 "10uF" V 5620 6505 50  0000 C CNN
 F 2 "" H 5820 6505 50  0001 C CNN
 F 3 "~" H 5820 6505 50  0001 C CNN
@@
 F 2 "Package_LGA:LGA-14_2x2mm_P0.35mm_LayoutBorder3x4y" H 4945 6355 50  0001 C CNN
 F 3 "" H 4945 6355 50  0001 C CNN
+F 4 "LIS2DHTR" H 4945 6355 50  0001 C CNN "Part Number"
 	1    4945 6355
 	1    0    0    -1
@@
 F 2 "Battery:BatteryHolder_MPD_BC2003_1x2032" V 10070 1620 50  0001 C CNN
 F 3 "~" V 10070 1620 50  0001 C CNN
+F 4 "CR2032R-HE1" H 10070 1560 50  0001 C CNN "Part Number"
 	1    10070 1560
 	1    0    0    -1
@@
 F 2 "Battery:BatteryHolder_MPD_BC2003_1x2032" V 8430 1620 50  0001 C CNN
 F 3 "~" V 8430 1620 50  0001 C CNN
+F 4 "CR2032R-HE1" H 8430 1560 50  0001 C CNN "Part Number"
 	1    8430 1560
 	1    0    0    -1
@@
 F 2 "" H 3705 3330 50  0001 C CNN
 F 3 "" H 3705 3330 50  0001 C CNN
+F 4 "nRF52832-QFAB-R" H 3705 3330 50  0001 C CNN "Part Number"
 	1    3705 3330
 	1    0    0    -1
@@
 F 2 "antena_ble:2450AT18B100" H 2345 5695 50  0001 C CNN
 F 3 "~" H 2345 5695 50  0001 C CNN
+F 4 "2450AT18B100E" H 2345 5695 50  0001 C CNN "Part Number"
 	1    2345 5695
 	1    0    0    -1

Commit message: BOM
correções no BOM
Parts:
- C1, C10, C11, C12, C13, C14, C15, C16, C17, C2, C3, C4, C5, C6, C7, C8, C9: footprint (none) -> Capacitor_SMD:C_0402_1005Metric
- L1, L3, L4, L5: footprint (none) -> Inductor_SMD:L_0402_1005Metric
- L2: value 10nH -> 10uH; footprint (none) -> Inductor_SMD:L_0402_1005Metric
- Y1: footprint (none) -> Crystal:Crystal_SMD_2016-4Pin_2.0x1.6mm
- Y2: footprint (none) -> Crystal:Crystal_SMD_3215-2Pin_3.2x1.5mm
Changed lines of the file:
@@
 F 0 "C4" H 2697 2176 50  0000 L CNN
 F 1 "4.7uF" H 2697 2085 50  0000 L CNN
-F 2 "" H 2605 2130 50  0001 C CNN
+F 2 "Capacitor_SMD:C_0402_1005Metric" H 2605 2130 50  0001 C CNN
 F 3 "~" H 2605 2130 50  0001 C CNN
 	1    2605 2130
@@
 F 0 "C1" H 3463 1384 50  0000 R CNN
 F 1 "1uF" H 3463 1475 50  0000 R CNN
-F 2 "" H 3555 1430 50  0001 C CNN
+F 2 "Capacitor_SMD:C_0402_1005Metric" H 3555 1430 50  0001 C CNN
 F 3 "~" H 3555 1430 50  0001 C CNN
 	1    3555 1430
@@
 F 0 "L1" H 3103 1476 50  0000 L CNN
 F 1 "15nH" H 3103 1385 50  0000 L CNN
-F 2 "" H 3055 1430 50  0001 C CNN
+F 2 "Inductor_SMD:L_0402_1005Metric" H 3055 1430 50  0001 C CNN
 F 3 "~" H 3055 1430 50  0001 C CNN
 	1    3055 1430
@@
 P 3055 1680
 F 0 "L2" H 3103 1726 50  0000 L CNN
-F 1 "10nH" H 3103 1635 50  0000 L CNN
-F 2 "" H 3055 1680 50  0001 C CNN
+F 1 "10uH" H 3103 1635 50  0000 L CNN
+F 2 "Inductor_SMD:L_0402_1005Metric" H 3055 1680 50  0001 C CNN
 F 3 "~" H 3055 1680 50  0001 C CNN
 	1    3055 1680
@@
 F 0 "C6" H 2097 2426 50  0000 L CNN
 F 1 "100nF" H 2097 2335 50  0000 L CNN
-F 2 "" H 2005 2380 50  0001 C CNN
+F 2 "Capacitor_SMD:C_0402_1005Metric" H 2005 2380 50  0001 C CNN
 F 3 "~" H 2005 2380 50  0001 C CNN
 	1    2005 2380
@@
 F 0 "C9" V 1026 2730 50  0000 C CNN
 F 1 "12pF" V 1117 2730 50  0000 C CNN
-F 2 "" H 1255 2730 50  0001 C CNN
+F 2 "Capacitor_SMD:C_0402_1005Metric" H 1255 2730 50  0001 C CNN
 F 3 "~" H 1255 2730 50  0001 C CNN
 	1    1255 2730
@@
 F 0 "Y2" V 1459 3018 50  0000 L CNN
 F 1 "32.768kHz" V 1550 3018 50  0000 L CNN
-F 2 "" H 1505 2930 50  0001 C CNN
+F 2 "Crystal:Crystal_SMD_3215-2Pin_3.2x1.5mm" H 1505 2930 50  0001 C CNN
 F 3 "~" H 1505 2930 50  0001 C CNN
 	1    1505 2930
@@
 F 0 "C11" V 1026 3130 50  0000 C CNN
 F 1 "12pF" V 1117 3130 50  0000 C CNN
-F 2 "" H 1255 3130 50  0001 C CNN
+F 2 "Capacitor_SMD:C_0402_1005Metric" H 1255 3130 50  0001 C CNN
 F 3 "~" H 1255 3130 50  0001 C CNN
 	1    1255 3130
@@
 F 0 "C14" H 2647 4526 50  0000 L CNN
 F 1 "100nF" H 2647 4435 50  0000 L CNN
-F 2 "" H 2555 4480 50  0001 C CNN
+F 2 "Capacitor_SMD:C_0402_1005Metric" H 2555 4480 50  0001 C CNN
 F 3 "~" H 2555 4480 50  0001 C CNN
 	1    2555 4480
@@
 F 0 "C7" H 4947 2526 50  0000 L CNN
 F 1 "100nF" H 4947 2435 50  0000 L CNN
-F 2 "" H 4855 2480 50  0001 C CNN
+F 2 "Capacitor_SMD:C_0402_1005Metric" H 4855 2480 50  0001 C CNN
 F 3 "~" H 4855 2480 50  0001 C CNN
 	1    4855 2480
@@
 F 0 "C5" V 5726 2280 50  0000 C CNN
 F 1 "12pF" V 5817 2280 50  0000 C CNN
-F 2 "" H 5955 2280 50  0001 C CNN
+F 2 "Capacitor_SMD:C_0402_1005Metric" H 5955 2280 50  0001 C CNN
 F 3 "~" H 5955 2280 50  0001 C CNN
 	1    5955 2280
@@
 F 0 "C8" V 5726 2680 50  0000 C CNN
 F 1 "12pF" V 5817 2680 50  0000 C CNN
-F 2 "" H 5955 2680 50  0001 C CNN
+F 2 "Capacitor_SMD:C_0402_1005Metric" H 5955 2680 50  0001 C CNN
 F 3 "~" H 5955 2680 50  0001 C CNN
 	1    5955 2680
@@
 F 0 "Y1" V 5709 2568 50  0000 L CNN
 F 1 "32MHz" V 5800 2568 50  0000 L CNN
-F 2 "" H 5755 2480 50  0001 C CNN
+F 2 "Crystal:Crystal_SMD_2016-4Pin_2.0x1.6mm" H 5755 2480 50  0001 C CNN
 F 3 "~" H 5755 2480 50  0001 C CNN
 	1    5755 2480
@@
 F 0 "C10" V 6181 2960 50  0000 C CNN
 F 1 "100pF" V 6272 2960 50  0000 C CNN
-F 2 "" H 6410 2960 50  0001 C CNN
+F 2 "Capacitor_SMD:C_0402_1005Metric" H 6410 2960 50  0001 C CNN
 F 3 "~" H 6410 2960 50  0001 C CNN
 	1    6410 2960
@@
 F 0 "C12" V 6181 3310 50  0000 C CNN
 F 1 "N.C." V 6272 3310 50  0000 C CNN
-F 2 "" H 6410 3310 50  0001 C CNN
+F 2 "Capacitor_SMD:C_0402_1005Metric" H 6410 3310 50  0001 C CNN
 F 3 "~" H 6410 3310 50  0001 C CNN
 	1    6410 3310
@@
 F 0 "C13" H 5547 3711 50  0000 L CNN
 F 1 "0.8pF" H 5547 3620 50  0000 L CNN
-F 2 "" H 5455 3665 50  0001 C CNN
+F 2 "Capacitor_SMD:C_0402_1005Metric" H 5455 3665 50  0001 C CNN
 F 3 "~" H 5455 3665 50  0001 C CNN
 	1    5455 3665
@@
 F 0 "L3" V 5595 3380 50  0000 C CNN
 F 1 "3.9nH" V 5530 3380 50  0000 C CNN
-F 2 "" H 5650 3380 50  0001 C CNN
+F 2 "Inductor_SMD:L_0402_1005Metric" H 5650 3380 50  0001 C CNN
 F 3 "~" H 5650 3380 50  0001 C CNN
 	1    5650 3380
@@
 F 0 "C17" V 5700 6840 50  0000 C CNN
 F 1 "100nF" V 5630 6840 50  0000 C CNN
-F 2 "" H 5830 6840 50  0001 C CNN
+F 2 "Capacitor_SMD:C_0402_1005Metric" H 5830 6840 50  0001 C CNN
 F 3 "~" H 5830 6840 50  0001 C CNN
 	1    5830 6840
@@
 F 0 "C16" V 5690 6505 50  0000 C CNN
 F 1 "10uF" V 5620 6505 50  0000 C CNN
-F 2 "" H 5820 6505 50  0001 C CNN
+F 2 "Capacitor_SMD:C_0402_1005Metric" H 5820 6505 50  0001 C CNN
 F 3 "~" H 5820 6505 50  0001 C CNN
 	1    5820 6505
@@
 F 0 "C3" H 9637 1551 50  0000 L CNN
 F 1 "1uF" H 9637 1460 50  0000 L CNN
-F 2 "" H 9545 1505 50  0001 C CNN
+F 2 "Capacitor_SMD:C_0402_1005Metric" H 9545 1505 50  0001 C CNN
 F 3 "~" H 9545 1505 50  0001 C CNN
 	1    9545 1505
@@
 F 0 "C2" H 7997 1551 50  0000 L CNN
 F 1 "1uF" H 7997 1460 50  0000 L CNN
-F 2 "" H 7905 1505 50  0001 C CNN
+F 2 "Capacitor_SMD:C_0402_1005Metric" H 7905 1505 50  0001 C CNN
 F 3 "~" H 7905 1505 50  0001 C CNN
 	1    7905 1505
@@
 F 0 "C15" V 1301 5905 50  0000 C CNN
 F 1 "1.2pF" V 1392 5905 50  0000 C CNN
-F 2 "" H 1530 5905 50  0001 C CNN
+F 2 "Capacitor_SMD:C_0402_1005Metric" H 1530 5905 50  0001 C CNN
 F 3 "~" H 1530 5905 50  0001 C CNN
 	1    1530 5905
@@
 F 0 "L5" H 1858 6096 50  0000 L CNN
 F 1 "2.7nH" H 1858 6005 50  0000 L CNN
-F 2 "" H 1810 6050 50  0001 C CNN
+F 2 "Inductor_SMD:L_0402_1005Metric" H 1810 6050 50  0001 C CNN
 F 3 "~" H 1810 6050 50  0001 C CNN
 	1    1810 6050
@@
 F 0 "L4" V 2235 5905 50  0000 C CNN
 F 1 "3.3nH" V 2144 5905 50  0000 C CNN
-F 2 "" H 2050 5905 50  0001 C CNN
+F 2 "Inductor_SMD:L_0402_1005Metric" H 2050 5905 50  0001 C CNN
 F 3 "~" H 2050 5905 50  0001 C CNN
 	1    2050 5905

Commit message: Resistores
resistências ajustadas, considerando agora a tensão do led

r = (v_bateria - v_led) / i_led
Parts:
- removed BT2: Battery_Cell, Battery:BatteryHolder_MPD_BC2003_1x2032, symbol Device:Battery_Cell
- removed C3: 1uF, Capacitor_SMD:C_0402_1005Metric, symbol Device:C_Small
- R1, R2, R3: value 100 -> 33
Connections:
- net VDD: now also R1.2, R2.2, R3.2, R4.1, R5.1, R6.1
- removed net VCC: R1.2, R2.2, R3.2, R4.1, R5.1, R6.1, U1.7 (Vdd_IO)
- no-connect marks 18 -> 19
Other:
- moved on the sheet: BT1, C2
Changed lines of the file:
@@
 Connection ~ 6610 3310
-$Comp
-L power:VCC #PWR018
-U 1 1 5E5B22F3
-P 9650 4685
-F 0 "#PWR018" H 9650 4535 50  0001 C CNN
-F 1 "VCC" H 9668 4858 50  0000 C CNN
-F 2 "" H 9650 4685 50  0001 C CNN
-F 3 "" H 9650 4685 50  0001 C CNN
-	1    9650 4685
-	1    0    0    -1
-$EndComp
 $Comp
 L Device:R_Small_US R4
@@
 	9650 4740 9650 4685
 $Comp
-L power:VCC #PWR020
-U 1 1 5E64A319
-P 8880 4705
-F 0 "#PWR020" H 8880 4555 50  0001 C CNN
-F 1 "VCC" H 8898 4878 50  0000 C CNN
-F 2 "" H 8880 4705 50  0001 C CNN
-F 3 "" H 8880 4705 50  0001 C CNN
-	1    8880 4705
-	1    0    0    -1
-$EndComp
-$Comp
 L Device:R_Small_US R6
 U 1 1 5E64A31F
@@
 	8880 4760 8880 4705
 $Comp
-L power:VCC #PWR019
-U 1 1 5E64D533
-P 8055 4690
-F 0 "#PWR019" H 8055 4540 50  0001 C CNN
-F 1 "VCC" H 8073 4863 50  0000 C CNN
-F 2 "" H 8055 4690 50  0001 C CNN
-F 3 "" H 8055 4690 50  0001 C CNN
-	1    8055 4690
-	1    0    0    -1
-$EndComp
-$Comp
 L Device:R_Small_US R5
 U 1 1 5E64D539
@@
 	8055 5475 8055 5450
 Wire Wire Line
-	8055 4745 8055 4690
-Wire Wire Line
 	8880 5065 8880 5045
 Text GLabel 7815 5040 0    50   Input ~ 0
@@
 P 8805 2925
 F 0 "R2" H 8873 2971 50  0000 L CNN
-F 1 "100" H 8873 2880 50  0000 L CNN
+F 1 "33" H 8873 2880 50  0000 L CNN
 F 2 "Resistor_SMD:R_0402_1005Metric" H 8805 2925 50  0001 C CNN
 F 3 "~" H 8805 2925 50  0001 C CNN
@@
 P 8065 2950
 F 0 "R3" H 8133 2996 50  0000 L CNN
-F 1 "100" H 8133 2905 50  0000 L CNN
+F 1 "33" H 8133 2905 50  0000 L CNN
 F 2 "Resistor_SMD:R_0402_1005Metric" H 8065 2950 50  0001 C CNN
 F 3 "~" H 8065 2950 50  0001 C CNN
@@
 P 9615 2910
 F 0 "R1" H 9683 2956 50  0000 L CNN
-F 1 "100" H 9683 2865 50  0000 L CNN
+F 1 "33" H 9683 2865 50  0000 L CNN
 F 2 "Resistor_SMD:R_0402_1005Metric" H 9615 2910 50  0001 C CNN
 F 3 "~" H 9615 2910 50  0001 C CNN
@@
 Wire Wire Line
 	8805 2825 8805 2765
-$Comp
-L power:VCC #PWR012
-U 1 1 5E59CC10
-P 8065 2790
-F 0 "#PWR012" H 8065 2640 50  0001 C CNN
-F 1 "VCC" H 8083 2963 50  0000 C CNN
-F 2 "" H 8065 2790 50  0001 C CNN
-F 3 "" H 8065 2790 50  0001 C CNN
-	1    8065 2790
-	1    0    0    -1
-$EndComp
-$Comp
-L power:VCC #PWR011
-U 1 1 5E59B1B1
-P 8805 2765
-F 0 "#PWR011" H 8805 2615 50  0001 C CNN
-F 1 "VCC" H 8823 2938 50  0000 C CNN
-F 2 "" H 8805 2765 50  0001 C CNN
-F 3 "" H 8805 2765 50  0001 C CNN
-	1    8805 2765
-	1    0    0    -1
-$EndComp
-$Comp
-L power:VCC #PWR010
-U 1 1 5E584D52
-P 9615 2750
-F 0 "#PWR010" H 9615 2600 50  0001 C CNN
-F 1 "VCC" H 9633 2923 50  0000 C CNN
-F 2 "" H 9615 2750 50  0001 C CNN
-F 3 "" H 9615 2750 50  0001 C CNN
-	1    9615 2750
-	1    0    0    -1
-$EndComp
 Wire Wire Line
 	9615 2810 9615 2750
@@
 $EndComp
 $Comp
-L power:VCC #PWR028
-U 1 1 5E803D5E
-P 5045 6905
-F 0 "#PWR028" H 5045 6755 50  0001 C CNN
-F 1 "VCC" H 5063 7078 50  0000 C CNN
-F 2 "" H 5045 6905 50  0001 C CNN
-F 3 "" H 5045 6905 50  0001 C CNN
-	1    5045 6905
-	-1   0    0    1
-$EndComp
-$Comp
 L power:Earth #PWR027
 U 1 1 5E7D824E
@@
 Wire Wire Line
 	4845 5615 4945 5615
-Text GLabel 9545 1360 0    50   Input ~ 0
-VCC
-Text GLabel 7905 1360 0    50   Input ~ 0
+Text GLabel 8770 1330 0    50   Input ~ 0
 VDD
-Connection ~ 10070 1730
-Wire Wire Line
-	10070 1730 10070 1660
-Wire Wire Line
-	9545 1730 10070 1730
-Wire Wire Line
-	9545 1605 9545 1730
-Wire Wire Line
-	9545 1360 9545 1405
-Wire Wire Line
-	10070 1360 9545 1360
-$Comp
-L power:Earth #PWR03
-U 1 1 5E6CCBBD
-P 10070 1730
-F 0 "#PWR03" H 10070 1480 50  0001 C CNN
-F 1 "Earth" H 10070 1580 50  0001 C CNN
-F 2 "" H 10070 1730 50  0001 C CNN
-F 3 "~" H 10070 1730 50  0001 C CNN
-	1    10070 1730
-	1    0    0    -1
-$EndComp
-$Comp
-L Device:C_Small C3
-U 1 1 5E6CCBB7
-P 9545 1505
-F 0 "C3" H 9637 1551 50  0000 L CNN
-F 1 "1uF" H 9637 1460 50  0000 L CNN
-F 2 "Capacitor_SMD:C_0402_1005Metric" H 9545 1505 50  0001 C CNN
-F 3 "~" H 9545 1505 50  0001 C CNN
-	1    9545 1505
-	1    0    0    -1
-$EndComp
-$Comp
-L Device:Battery_Cell BT2
-U 1 1 5E6CCBB1
-P 10070 1560
-F 0 "BT2" H 10188 1656 50  0000 L CNN
-F 1 "Battery_Cell" H 10188 1565 50  0000 L CNN
-F 2 "Battery:BatteryHolder_MPD_BC2003_1x2032" V 10070 1620 50  0001 C CNN
-F 3 "~" V 10070 1620 50  0001 C CNN
-F 4 "CR2032R-HE1" H 10070 1560 50  0001 C CNN "Part Number"
-	1    10070 1560
-	1    0    0    -1
-$EndComp
-Connection ~ 8430 1730
-Wire Wire Line
-	8430 1730 8430 1660
-Wire Wire Line
-	7905 1730 8430 1730
-Wire Wire Line
-	7905 1605 7905 1730
-Wire Wire Line
-	7905 1360 7905 1405
-Wire Wire Line
-	8430 1360 7905 1360
+Connection ~ 9295 1700
+Wire Wire Line
+	9295 1700 9295 1630
+Wire Wire Line
+	8770 1700 9295 1700
+Wire Wire Line
+	8770 1575 8770 1700
+Wire Wire Line
+	8770 1330 8770 1375
+Wire Wire Line
+	9295 1330 8770 1330
 $Comp
 L power:Earth #PWR02
 U 1 1 5E6C4346
-P 8430 1730
-F 0 "#PWR02" H 8430 1480 50  0001 C CNN
-F 1 "Earth" H 8430 1580 50  0001 C CNN
-F 2 "" H 8430 1730 50  0001 C CNN
-F 3 "~" H 8430 1730 50  0001 C CNN
-	1    8430 1730
+P 9295 1700
+F 0 "#PWR02" H 9295 1450 50  0001 C CNN
+F 1 "Earth" H 9295 1550 50  0001 C CNN
+F 2 "" H 9295 1700 50  0001 C CNN
+F 3 "~" H 9295 1700 50  0001 C CNN
+	1    9295 1700
 	1    0    0    -1
 $EndComp
@@
 L Device:C_Small C2
 U 1 1 5E6BE474
-P 7905 1505
-F 0 "C2" H 7997 1551 50  0000 L CNN
-F 1 "1uF" H 7997 1460 50  0000 L CNN
-F 2 "Capacitor_SMD:C_0402_1005Metric" H 7905 1505 50  0001 C CNN
-F 3 "~" H 7905 1505 50  0001 C CNN
-	1    7905 1505
+P 8770 1475
+F 0 "C2" H 8862 1521 50  0000 L CNN
+F 1 "1uF" H 8862 1430 50  0000 L CNN
+F 2 "Capacitor_SMD:C_0402_1005Metric" H 8770 1475 50  0001 C CNN
+F 3 "~" H 8770 1475 50  0001 C CNN
+	1    8770 1475
 	1    0    0    -1
 $EndComp
@@
 L Device:Battery_Cell BT1
 U 1 1 5E6BC499
-P 8430 1560
-F 0 "BT1" H 8548 1656 50  0000 L CNN
-F 1 "Battery_Cell" H 8548 1565 50  0000 L CNN
-F 2 "Battery:BatteryHolder_MPD_BC2003_1x2032" V 8430 1620 50  0001 C CNN
-F 3 "~" V 8430 1620 50  0001 C CNN
-F 4 "CR2032R-HE1" H 8430 1560 50  0001 C CNN "Part Number"
-	1    8430 1560
+P 9295 1530
+F 0 "BT1" H 9413 1626 50  0000 L CNN
+F 1 "Battery_Cell" H 9413 1535 50  0000 L CNN
+F 2 "Battery:BatteryHolder_MPD_BC2003_1x2032" V 9295 1590 50  0001 C CNN
+F 3 "~" V 9295 1590 50  0001 C CNN
+F 4 "CR2032R-HE1" H 9295 1530 50  0001 C CNN "Part Number"
+	1    9295 1530
 	1    0    0    -1
 $EndComp
@@
 Wire Notes Line
 	3005 6510 3005 7645
+$Comp
+L power:VDD #PWR?
+U 1 1 5E5987B3
+P 8065 2790
+F 0 "#PWR?" H 8065 2640 50  0001 C CNN
+F 1 "VDD" H 8082 2963 50  0000 C CNN
+F 2 "" H 8065 2790 50  0001 C CNN
+F 3 "" H 8065 2790 50  0001 C CNN
+	1    8065 2790
+	1    0    0    -1
+$EndComp
+$Comp
+L power:VDD #PWR?
+U 1 1 5E59EF9F
+P 8805 2765
+F 0 "#PWR?" H 8805 2615 50  0001 C CNN
+F 1 "VDD" H 8822 2938 50  0000 C CNN
+F 2 "" H 8805 2765 50  0001 C CNN
+F 3 "" H 8805 2765 50  0001 C CNN
+	1    8805 2765
+	1    0    0    -1
+$EndComp
+$Comp
+L power:VDD #PWR?
+U 1 1 5E5A4F33
+P 9615 2750
+F 0 "#PWR?" H 9615 2600 50  0001 C CNN
+F 1 "VDD" H 9632 2923 50  0000 C CNN
+F 2 "" H 9615 2750 50  0001 C CNN
+F 3 "" H 9615 2750 50  0001 C CNN
+	1    9615 2750
+	1    0    0    -1
+$EndComp
+Wire Wire Line
+	8055 4745 8055 4690
+$Comp
+L power:VDD #PWR?
+U 1 1 5E5B249E
+P 8055 4690
+F 0 "#PWR?" H 8055 4540 50  0001 C CNN
+F 1 "VDD" H 8072 4863 50  0000 C CNN
+F 2 "" H 8055 4690 50  0001 C CNN
+F 3 "" H 8055 4690 50  0001 C CNN
+	1    8055 4690
+	1    0    0    -1
+$EndComp
+$Comp
+L power:VDD #PWR?
+U 1 1 5E5B8527
+P 8880 4705
+F 0 "#PWR?" H 8880 4555 50  0001 C CNN
+F 1 "VDD" H 8897 4878 50  0000 C CNN
+F 2 "" H 8880 4705 50  0001 C CNN
+F 3 "" H 8880 4705 50  0001 C CNN
+	1    8880 4705
+	1    0    0    -1
+$EndComp
+$Comp
+L power:VDD #PWR?
+U 1 1 5E5BE646
+P 9650 4685
+F 0 "#PWR?" H 9650 4535 50  0001 C CNN
+F 1 "VDD" H 9667 4858 50  0000 C CNN
+F 2 "" H 9650 4685 50  0001 C CNN
+F 3 "" H 9650 4685 50  0001 C CNN
+	1    9650 4685
+	1    0    0    -1
+$EndComp
+NoConn ~ 5045 6905
 $EndSCHEMATC
