File: BKR01AT/BKR01AT.sch (KiCad schematic (older format))
At the start: 44 parts, among them J1 Conn_02x03_Odd_Even, SW1 SW_Push, SW2 SW_Push, SW3 SW_Push, U1 LIS2DHTR, Y1 32MHz, Y2 32.768kHz

Commit message: gerbers
Connections:
- wire segments 137 -> 132
Other:
- moved on the sheet: AE1, C15, L4, L5
